File: bot_board/bot_board/bot_board.kicad_pcb (KiCad board)
At the start: 2 copper layers, 62 x 81 mm, 15 parts, among them J1 ENCODER, J10 ENCODER, J11 ENCODER, J2 PROG, J3 MISC, J4 POWER, J5 5V, J6 GND, J7 3V3, J8 GPS+OLED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

Commit message: Bot board done. Pow board started
Parts:
- added C1: 100n, Capacitor_SMD:C_1206_3216Metric_Pad1.33x1.80mm_HandSolder, B.Cu at (109.8, 125.5)
- added C2: 100n, Capacitor_SMD:C_1206_3216Metric_Pad1.33x1.80mm_HandSolder, B.Cu at (109.9, 117.8)
- added C3: 100n, Capacitor_SMD:C_1206_3216Metric_Pad1.33x1.80mm_HandSolder, B.Cu at (109.9, 120.4)
- added C4: 100n, Capacitor_SMD:C_1206_3216Metric_Pad1.33x1.80mm_HandSolder, B.Cu at (72.1, 118.6)
- added C5: 100n, Capacitor_SMD:C_1206_3216Metric_Pad1.33x1.80mm_HandSolder, B.Cu at (89.2, 136.9)
- added C6: 100u, Capacitor_Tantalum_SMD:CP_EIA-3528-21_Kemet-B_Pad1.50x2.35mm_HandSolder, B.Cu at (92.3, 135.3)
- added C7: 100n, Capacitor_SMD:C_1206_3216Metric_Pad1.33x1.80mm_HandSolder, B.Cu at (86.9, 136.8)
- added J12: BUTTON, Connector_PinHeader_2.54mm:PinHeader_1x02_P2.54mm_Horizontal, F.Cu at (74.7, 117.6)
- added J13: OLED, Connector_PinHeader_2.54mm:PinHeader_1x04_P2.54mm_Horizontal, F.Cu at (102.3, 131.2)
- added J14: GPS, Connector_PinHeader_2.54mm:PinHeader_1x04_P2.54mm_Horizontal, F.Cu at (91.1, 131.2)
- added J15: POWER IN, Connector_PinHeader_2.54mm:PinHeader_1x05_P2.54mm_Horizontal, F.Cu at (74.8, 85.7)
- added R1: 10k, Resistor_SMD:R_1206_3216Metric_Pad1.30x1.75mm_HandSolder, B.Cu at (119.7, 125.7)
- added R10: 10k, Resistor_SMD:R_1206_3216Metric_Pad1.30x1.75mm_HandSolder, B.Cu at (72.1, 113.6)
- added R11: 57K6, Resistor_SMD:R_1210_3225Metric_Pad1.30x2.65mm_HandSolder, B.Cu at (79.5, 86.0)
- added R12: 110K, Resistor_SMD:R_1206_3216Metric_Pad1.30x1.75mm_HandSolder, B.Cu at (82.6, 83.1)
- added R13: 0R, Resistor_SMD:R_1206_3216Metric_Pad1.30x1.75mm_HandSolder, B.Cu at (87.7, 107.2)
- added R14: 0R, Resistor_SMD:R_1206_3216Metric_Pad1.30x1.75mm_HandSolder, B.Cu at (70.7, 96.2)
- added R15: 0R, Resistor_SMD:R_1206_3216Metric_Pad1.30x1.75mm_HandSolder, B.Cu at (84.8, 90.6)
- added R2: 10k, Resistor_SMD:R_1206_3216Metric_Pad1.30x1.75mm_HandSolder, B.Cu at (109.9, 123.0)
- added R3: 10k, Resistor_SMD:R_1206_3216Metric_Pad1.30x1.75mm_HandSolder, B.Cu at (115.0, 135.2)
- added R4: 10k, Resistor_SMD:R_1206_3216Metric_Pad1.30x1.75mm_HandSolder, B.Cu at (124.9, 125.7)
- added R5: 10k, Resistor_SMD:R_1206_3216Metric_Pad1.30x1.75mm_HandSolder, B.Cu at (112.5, 135.2)
- added R6: 10k, Resistor_SMD:R_1206_3216Metric_Pad1.30x1.75mm_HandSolder, B.Cu at (122.3, 125.7)
- added R7: 100k, Resistor_SMD:R_1210_3225Metric_Pad1.30x2.65mm_HandSolder, B.Cu at (79.2, 78.2)
- added R8: 10k, Resistor_SMD:R_1206_3216Metric_Pad1.30x1.75mm_HandSolder, B.Cu at (79.2, 75.3)
- added R9: 1k, Resistor_SMD:R_1206_3216Metric_Pad1.30x1.75mm_HandSolder, B.Cu at (96.2, 109.7)
- J10: value ENCODER -> UART
- J3: moved to F.Cu
- moved J11 15.2 mm to (115.1, 131.2), turned to -90 degrees
- moved J10 5.62 mm to (116.8, 105.5)
- turned J3 to 0 degrees
Connections:
- J11 pad 1: ENC_A -> ENC_O_A
- J11 pad 2: ENC_E -> ENC_O_E
- J11 pad 3: ENC_P -> ENC_O_P
Routing:
- net +3.3V: track 0.00 -> 152.6 mm
- net GND: track 0.00 -> 82.3 mm
- net Net-(R7-Pad1): track 0.00 -> 52.5 mm
- net EXT_POWER_DETECT: track 0.00 -> 28.6 mm
- net +5V: track 0.00 -> 26.4 mm
- net SDA: track 0.00 -> 22.6 mm
- net GPS_RX: track 0.00 -> 22.0 mm
- net BUTTON: track 0.00 -> 21.2 mm
- net SCL: track 0.00 -> 18.9 mm
- net ENC_O_A: track 0.00 -> 14.8 mm
- net ENC_O_E: track 0.00 -> 14.7 mm
- net ENC_O_P: track 0.00 -> 12.1 mm
- net ENC_A: track 8.17 -> 18.6 mm
- net BATTERY: track 0.00 -> 6.40 mm
- net RX0: track 8.30 -> 2.42 mm
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Other:
- board text added: "3 C D G"
- board text added: "B G"
- board text added: "B G 5 3 U"
- board text added: "G P E A"
- board text added: "G T R 3"
- board text added: "GT GR G 3"
- board text removed: "3V3"
- board text removed: "5V"
- board text removed: "BATT"
- board text removed: "BUTT"
- board text removed: "ENCA"
- board text removed: "ENCE"
- board text removed: "ENCP"
- board text removed: "EXTP"
- board text removed: "GND"
- board text removed: "GR"
- board text removed: "GT"
- board text removed: "SC"
- board text removed: "SD"
