File: bot_board/bot_board/bot_board.kicad_sch (KiCad schematic)
At the start: 35 parts, among them J1 ENCODER, J10 UART, J11 ENCODER, J12 BUTTON, J13 OLED, J14 GPS, J2 PROG, J3 MISC, J4 POWER, J5 5V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

Commit message: Bot board done. Pow board started
Parts:
- added J15: POWER IN, Connector_PinHeader_2.54mm:PinHeader_1x05_P2.54mm_Horizontal, symbol Connector:Conn_01x05_Pin
- added R11: 57K6, Resistor_SMD:R_1210_3225Metric_Pad1.30x2.65mm_HandSolder, symbol Device:R
- added R12: 110K, Resistor_SMD:R_1206_3216Metric_Pad1.30x1.75mm_HandSolder, symbol Device:R
- added R13, R14, R15: 0R, Resistor_SMD:R_1206_3216Metric_Pad1.30x1.75mm_HandSolder, symbol Device:R
Connections:
- net +3.3V: now also J14.1 (Pin_1), J15.2 (Pin_2); no longer J14.4 (Pin_4)
- net +5V: now also J15.3 (Pin_3)
- net +BATT: now also J15.5 (Pin_5)
- net ENC_O_P: no longer C1.1, R1.1, R2.1
- net ENC_P: now also C1.1, R1.1, R2.1
- net EXT_POWER_DETECT: now also R11.1, R12.2, R13.1, R13.2
- net GND: now also J14.2 (Pin_2), J15.4 (Pin_4), R12.1, R14.1, R14.2, R15.1, R15.2; no longer J14.1 (Pin_1)
- net GPS_RX: now also J14.3 (Pin_3); no longer J14.2 (Pin_2)
- net GPS_TX: now also J14.4 (Pin_4); no longer J14.3 (Pin_3)
- net SCL: now also J13.3 (Pin_3); no longer J13.2 (Pin_2)
- net SDA: now also J13.2 (Pin_2); no longer J13.3 (Pin_3)
- new net VBUS: J15.1 (Pin_1), R11.2
Other:
- moved on the sheet: C5, C6, C7, J10, J13, J14, J2, J4, J5, J6, J7, J8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
