File: pow_board/pow_board/pow_board.kicad_pcb (KiCad board)
At the start: 2 copper layers, 62 x 81 mm, 5 parts, among them J1 POWER IN

Commit message: pow board start
Parts:
- added BT1: Battery_Cell, Battery:BatteryHolder_Keystone_1042_1x18650, F.Cu at (87.1, 100.8)
- added C1: 100n, Capacitor_SMD:C_1206_3216Metric_Pad1.33x1.80mm_HandSolder, F.Cu at (143.4, 95.7)
- added C2: 22u, Capacitor_SMD:C_1206_3216Metric_Pad1.33x1.80mm_HandSolder, F.Cu at (143.4, 99.0)
- added C4: 100n, Capacitor_SMD:C_1206_3216Metric_Pad1.33x1.80mm_HandSolder, F.Cu at (143.4, 102.4)
- added C5: 22u, Capacitor_SMD:C_1206_3216Metric_Pad1.33x1.80mm_HandSolder, F.Cu at (143.4, 105.7)
- added J2: EXT_USB, Connector_PinSocket_2.54mm:PinSocket_1x02_P2.54mm_Horizontal, F.Cu at (130.8, 68.1)
- added J3: EXT_BAT, Connector_PinSocket_2.54mm:PinSocket_1x02_P2.54mm_Horizontal, F.Cu at (130.8, 75.2)
- added R1: 0R, Resistor_SMD:R_1206_3216Metric_Pad1.30x1.75mm_HandSolder, F.Cu at (149.4, 102.8)
- added SW1: SW_SPST, Connector_PinHeader_2.54mm:PinHeader_1x02_P2.54mm_Horizontal, F.Cu at (148.8, 96.3)
- added U1: Battery charger module, 0a_pow:TP4056_module_typeC, F.Cu at (46.4, 95.3)
- added U2: Step-up DC-DC, 0a_pow:MT3608_step-up_DC-DC, B.Cu at (70.7, 90.5)
Connections:
- J1 pad 1: (no net) -> VBUS
- J1 pad 2: (no net) -> +3.3V
- J1 pad 3: (no net) -> +5V
- J1 pad 4: (no net) -> GND
- J1 pad 5: (no net) -> +BATT
Other:
- board size 62 x 81 mm -> 62 x 89.4 mm
