File: pow_board/pow_board/pow_board.kicad_sch (KiCad schematic)
At the start: 1 part, among them J1 POWER IN

Commit message: pow board start
Parts:
- added BT1: Battery_Cell, Battery:BatteryHolder_Keystone_1042_1x18650, symbol Device:Battery_Cell
- added C1, C4: 100n, Capacitor_SMD:C_1206_3216Metric_Pad1.33x1.80mm_HandSolder, symbol Device:C
- added C2, C5: 22u, Capacitor_SMD:C_1206_3216Metric_Pad1.33x1.80mm_HandSolder, symbol Device:C
- added H1, H2, H3, H4: MountingHole, MountingHole:MountingHole_3.2mm_M3, symbol Mechanical:MountingHole
- added J2: EXT_USB, Connector_PinSocket_2.54mm:PinSocket_1x02_P2.54mm_Horizontal, symbol Connector:Conn_01x02_Pin
- added J3: EXT_BAT, Connector_PinSocket_2.54mm:PinSocket_1x02_P2.54mm_Horizontal, symbol Connector:Conn_01x02_Pin
- added R1: 0R, Resistor_SMD:R_1206_3216Metric_Pad1.30x1.75mm_HandSolder, symbol Device:R
- added SW1: SW_SPST, Connector_PinHeader_2.54mm:PinHeader_1x02_P2.54mm_Horizontal, symbol Switch:SW_SPST
- added U1: Battery charger module, 0a_pow:TP4056_module_typeC, symbol 0a_pow:TP4056_module_typeC
- added U2: Step-up DC-DC, 0a_pow:MT3608_step-up_DC-DC, symbol 0a_pow:MT3608_step-up_DC-DC
- added U3: Step-down DC-DC, symbol 0a_pow:LM2596 step-down DC-DC module
Connections:
- net +3.3V: now also C4.1, C5.1, U3. (OUT-)
- net +5V: now also C1.1, C2.1, U2.3 (OUT+), U3.1 (IN+)
- net +BATT: now also BT1.1 (+), J3.2 (Pin_2), U1.5 (BAT+)
- net GND: now also BT1.2 (-), C1.2, C2.2, C4.2, C5.2, J2.1 (Pin_1), J3.1 (Pin_1), R1.1, R1.2, U1.2 (USB-), U1.4 (OUT-), U1.6 (BAT-), U2.2 (IN-), U2.4 (OUT-), U3. (OUT-), U3.2 (IN-)
- net VBUS: now also J2.2 (Pin_2), U1.1 (USB+)
- new net: SW1.1 (A), U1.3 (OUT+)
- new net: SW1.2 (B), U2.1 (IN+)
Other:
- moved on the sheet: J1
