File: bot_board/bot_board.kicad_pcb (KiCad board)
At the start: 2 copper layers, 62 x 81 mm, 41 parts, among them J1 ENCODER, J10 UART, J11 ENCODER, J12 BUTTON, J13 OLED, J14 GPS, J15 POWER IN, J2 PROG, J3 MISC, J4 POWER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

Commit message: Boards done, composition done
Parts:
- J1, J8: footprint Connector_PinHeader_2.54mm:PinHeader_1x04_P2.54mm_Vertical -> Connector_PinSocket_2.54mm:PinSocket_1x04_P2.54mm_Vertical
- J2, J5, J6, J7: footprint Connector_PinHeader_2.54mm:PinHeader_1x02_P2.54mm_Vertical -> Connector_PinSocket_2.54mm:PinSocket_1x02_P2.54mm_Vertical
- J3, J4: footprint Connector_PinHeader_2.54mm:PinHeader_1x03_P2.54mm_Vertical -> Connector_PinSocket_2.54mm:PinSocket_1x03_P2.54mm_Vertical
- J9: footprint Connector_PinHeader_2.54mm:PinHeader_1x01_P2.54mm_Vertical -> Connector_PinSocket_2.54mm:PinSocket_1x01_P2.54mm_Vertical

Commit message: Recovering after git fatal error. Changed M3 to M4
Parts:
- H1, H2, H3, H4: footprint MountingHole:MountingHole_3.2mm_M3 -> MountingHole:MountingHole_4.3mm_M4
Other:
- board text added: "M4"
- board text removed: "M3"
Changed lines of the file:
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@@
 		)
 	)
-	(footprint "MountingHole:MountingHole_3.2mm_M3"
+	(footprint "MountingHole:MountingHole_4.3mm_M4"
 		(layer "F.Cu")
 		(at 69.65 64.56)
-		(descr "Mounting Hole 3.2mm, no annular, M3")
-		(tags "mounting hole 3.2mm no annular m3")
+		(descr "Mounting Hole 4.3mm, no annular, M4")
+		(tags "mounting hole 4.3mm no annular m4")
 		(property "Reference" "H1"
-			(at 0 -4.2 0)
+			(at 0 -5.3 0)
 			(layer "F.SilkS")
 			(hide yes)
@@
 		)
 		(property "Value" "MountingHole"
-			(at 0 4.2 0)
+			(at 0 5.3 0)
 			(layer "F.Fab")
-			(hide yes)
 			(effects
 				(font
@@
 			)
 		)
-		(property "Footprint" "MountingHole:MountingHole_3.2mm_M3"
+		(property "Footprint" "MountingHole:MountingHole_4.3mm_M4"
 			(at 0 0 0)
 			(unlocked yes)
@@
 		(fp_circle
 			(center 0 0)
-			(end 3.2 0)
+			(end 4.3 0)
 			(stroke
 				(width 0.15)
@@
 		(fp_circle
 			(center 0 0)
-			(end 3.45 0)
+			(end 4.55 0)
 			(stroke
 				(width 0.05)
@@
 		(pad "" np_thru_hole circle
 			(at 0 0)
-			(size 3.2 3.2)
-			(drill 3.2)
-			(layers "F&B.Cu" "*.Mask")
+			(size 4.3 4.3)
+			(drill 4.3)
+			(layers "*.Cu" "*.Mask")
 		)
 	)
-	(footprint "MountingHole:MountingHole_3.2mm_M3"
+	(footprint "MountingHole:MountingHole_4.3mm_M4"
 		(layer "F.Cu")
 		(at 69.65 135.56)
-		(descr "Mounting Hole 3.2mm, no annular, M3")
-		(tags "mounting hole 3.2mm no annular m3")
+		(descr "Mounting Hole 4.3mm, no annular, M4")
+		(tags "mounting hole 4.3mm no annular m4")
 		(property "Reference" "H3"
-			(at 0 -4.2 0)
+			(at 0 -5.3 0)
 			(layer "F.SilkS")
 			(hide yes)
@@
 		)
 		(property "Value" "MountingHole"
-			(at 0 4.2 0)
+			(at 0 5.3 0)
 			(layer "F.Fab")
-			(hide yes)
 			(effects
 				(font
@@
 			)
 		)
-		(property "Footprint" "MountingHole:MountingHole_3.2mm_M3"
+		(property "Footprint" "MountingHole:MountingHole_4.3mm_M4"
 			(at 0 0 0)
 			(unlocked yes)
@@
 		(fp_circle
 			(center 0 0)
-			(end 3.2 0)
+			(end 4.3 0)
 			(stroke
 				(width 0.15)
@@
 		(fp_circle
 			(center 0 0)
-			(end 3.45 0)
+			(end 4.55 0)
 			(stroke
 				(width 0.05)
@@
 		(pad "" np_thru_hole circle
 			(at 0 0)
-			(size 3.2 3.2)
-			(drill 3.2)
-			(layers "F&B.Cu" "*.Mask")
+			(size 4.3 4.3)
+			(drill 4.3)
+			(layers "*.Cu" "*.Mask")
 		)
 	)
@@
 		)
 	)
-	(footprint "MountingHole:MountingHole_3.2mm_M3"
+	(footprint "MountingHole:MountingHole_4.3mm_M4"
 		(layer "F.Cu")
 		(at 121.65 64.56)
-		(descr "Mounting Hole 3.2mm, no annular, M3")
-		(tags "mounting hole 3.2mm no annular m3")
+		(descr "Mounting Hole 4.3mm, no annular, M4")
+		(tags "mounting hole 4.3mm no annular m4")
 		(property "Reference" "H2"
-			(at 0 -4.2 0)
+			(at 0 -5.3 0)
 			(layer "F.SilkS")
 			(hide yes)
@@
 		)
 		(property "Value" "MountingHole"
-			(at 0 4.2 0)
+			(at 0 5.3 0)
 			(layer "F.Fab")
-			(hide yes)
 			(effects
 				(font
@@
 			)
 		)
-		(property "Footprint" "MountingHole:MountingHole_3.2mm_M3"
+		(property "Footprint" "MountingHole:MountingHole_4.3mm_M4"
 			(at 0 0 0)
 			(unlocked yes)
@@
 		(fp_circle
 			(center 0 0)
-			(end 3.2 0)
+			(end 4.3 0)
 			(stroke
 				(width 0.15)
@@
 		(fp_circle
 			(center 0 0)
-			(end 3.45 0)
+			(end 4.55 0)
 			(stroke
 				(width 0.05)
@@
 		(pad "" np_thru_hole circle
 			(at 0 0)
-			(size 3.2 3.2)
-			(drill 3.2)
-			(layers "F&B.Cu" "*.Mask")
+			(size 4.3 4.3)
+			(drill 4.3)
+			(layers "*.Cu" "*.Mask")
 		)
 	)
@@
 		)
 	)
-	(footprint "MountingHole:MountingHole_3.2mm_M3"
+	(footprint "MountingHole:MountingHole_4.3mm_M4"
 		(layer "F.Cu")
 		(at 121.65 135.56)
-		(descr "Mounting Hole 3.2mm, no annular, M3")
-		(tags "mounting hole 3.2mm no annular m3")
+		(descr "Mounting Hole 4.3mm, no annular, M4")
+		(tags "mounting hole 4.3mm no annular m4")
 		(property "Reference" "H4"
-			(at 0 -4.2 0)
+			(at 0 -5.3 0)
 			(layer "F.SilkS")
 			(hide yes)
@@
 		)
 		(property "Value" "MountingHole"
-			(at 0 4.2 0)
+			(at 0 5.3 0)
 			(layer "F.Fab")
-			(hide yes)
 			(effects
 				(font
@@
 			)
 		)
-		(property "Footprint" "MountingHole:MountingHole_3.2mm_M3"
+		(property "Footprint" "MountingHole:MountingHole_4.3mm_M4"
 			(at 0 0 0)
 			(unlocked yes)
@@
 		(fp_circle
 			(center 0 0)
-			(end 3.2 0)
+			(end 4.3 0)
 			(stroke
 				(width 0.15)
@@
 		(fp_circle
 			(center 0 0)
-			(end 3.45 0)
+			(end 4.55 0)
 			(stroke
 				(width 0.05)
@@
 		(pad "" np_thru_hole circle
 			(at 0 0)
-			(size 3.2 3.2)
-			(drill 3.2)
-			(layers "F&B.Cu" "*.Mask")
+			(size 4.3 4.3)
+			(drill 4.3)
+			(layers "*.Cu" "*.Mask")
 		)
 	)
@@
 		(layer "B.Fab")
 	)
-	(gr_text "M3"
-		(at 77.51 64.64 -0)
+	(gr_text "M4"
+		(at 78.22 64.22 0)
 		(layer "B.Cu")
 		(effects
@@
 	)
 	(gr_text "52X71MM"
-		(at 84.71 66.94 -0)
+		(at 85.42 66.52 -0)
 		(layer "B.Cu")
 		(effects
@@
 	)
 	(segment
-		(start 122.88 131.17)
-		(end 115 131.17)
+		(start 124.94 129.11)
+		(end 123.46 130.59)
 		(width 0.5)
 		(layer "B.Cu")
@@
 	)
 	(segment
-		(start 114.97 133.61)
-		(end 114.97 131.62)
+		(start 124.94 127.23)
+		(end 124.94 129.11)
 		(width 0.5)
 		(layer "B.Cu")
@@
 	)
 	(segment
-		(start 124.94 127.23)
-		(end 124.94 128.72)
+		(start 114.97 133.61)
+		(end 114.97 131.62)
 		(width 0.5)
 		(layer "B.Cu")
@@
 	)
 	(segment
-		(start 123.84 130.21)
-		(end 122.88 131.17)
-		(width 0.5)
-		(layer "B.Cu")
-		(net 18)
-	)
-	(segment
-		(start 124.94 128.72)
-		(end 124.94 129.11)
+		(start 115.58 130.59)
+		(end 115 131.17)
 		(width 0.5)
 		(layer "B.Cu")
@@
 	)
 	(segment
-		(start 124.94 129.11)
-		(end 123.84 130.21)
+		(start 123.46 130.59)
+		(end 115.58 130.59)
 		(width 0.5)
 		(layer "B.Cu")
