File: top_board/ld1.kicad_sch (KiCad schematic)
At the start: 45 parts, among them J1 ENCODER, J2 PROG, J3 MISC, J4 POWER, J5 5V, J6 GND, J7 3V3, J8 GPS+OLED, J9 GND, SW3 KLS7-KL-02-N-0-0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

Commit message: Recovering after git fatal error. Changed M3 to M4
Parts:
- H1, H2, H3, H4: footprint MountingHole:MountingHole_3.2mm_M3 -> MountingHole:MountingHole_4.3mm_M4
Changed lines of the file:
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@@
 			)
 		)
-		(property "Footprint" "MountingHole:MountingHole_3.2mm_M3"
+		(property "Footprint" "MountingHole:MountingHole_4.3mm_M4"
 			(at 219.71 113.03 0)
 			(effects
@@
 			)
 		)
-		(property "Footprint" "MountingHole:MountingHole_3.2mm_M3"
+		(property "Footprint" "MountingHole:MountingHole_4.3mm_M4"
 			(at 219.71 120.65 0)
 			(effects
@@
 			)
 		)
-		(property "Footprint" "MountingHole:MountingHole_3.2mm_M3"
+		(property "Footprint" "MountingHole:MountingHole_4.3mm_M4"
 			(at 219.71 129.54 0)
 			(effects
@@
 			)
 		)
-		(property "Footprint" "MountingHole:MountingHole_3.2mm_M3"
+		(property "Footprint" "MountingHole:MountingHole_4.3mm_M4"
 			(at 219.71 138.43 0)
 			(effects
