File: pow_board/pow_board.kicad_sch (KiCad schematic)
At the start: 17 parts, among them J1 POWER IN, J2 EXT_USB, J3 EXT_BAT, SW1 SW_SPST, U1 Battery charger module, U2 Step-up DC-DC, U3 Step-down DC-DC

Commit message: Boards done, composition done
Parts:
- J2, J3: footprint Connector_PinSocket_2.54mm:PinSocket_1x02_P2.54mm_Horizontal -> Connector_PinHeader_2.54mm:PinHeader_1x02_P2.54mm_Horizontal
- U3: footprint (none) -> 0a_pow:LM2596 step-down DC-DC module
Connections:
- net +3.3V: now also U3.3 (OUT+); no longer U3. (OUT-)
- net GND: now also U3.4 (OUT-); no longer R1.1, R1.2, U3. (OUT-)
- net VBUS: now also R1.1, R1.2
- net at SW1.1 (A): now also U2.1 (IN+); no longer U1.3 (OUT+)
- net at SW1.2 (B): now also U1.3 (OUT+); no longer U2.1 (IN+)

Commit message: Recovering after git fatal error. Changed M3 to M4
Parts:
- H1, H2, H3, H4: footprint MountingHole:MountingHole_3.2mm_M3 -> MountingHole:MountingHole_4.3mm_M4
Changed lines of the file:
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@@
 			)
 		)
-		(property "Footprint" "MountingHole:MountingHole_3.2mm_M3"
+		(property "Footprint" "MountingHole:MountingHole_4.3mm_M4"
 			(at 260.35 149.86 0)
 			(effects
@@
 			)
 		)
-		(property "Footprint" "MountingHole:MountingHole_3.2mm_M3"
+		(property "Footprint" "MountingHole:MountingHole_4.3mm_M4"
 			(at 260.35 140.97 0)
 			(effects
@@
 			)
 		)
-		(property "Footprint" "MountingHole:MountingHole_3.2mm_M3"
+		(property "Footprint" "MountingHole:MountingHole_4.3mm_M4"
 			(at 260.35 133.35 0)
 			(effects
@@
 			)
 		)
-		(property "Footprint" "MountingHole:MountingHole_3.2mm_M3"
+		(property "Footprint" "MountingHole:MountingHole_4.3mm_M4"
 			(at 260.35 158.75 0)
 			(effects

Commit message: Update
Parts:
- added D1: VS-15MQ040NTRPBF, Diode_SMD:D_SMA_Handsoldering, symbol Device:D_Schottky
- added Q1: IRLML6401, Package_TO_SOT_SMD:SOT-23, symbol Transistor_FET:IRLML6401
- added R2: 10k, Resistor_SMD:R_1206_3216Metric_Pad1.30x1.75mm_HandSolder, symbol Device:R
- added R3, R4, R5, R6: 0R, Resistor_SMD:R_1206_3216Metric_Pad1.30x1.75mm_HandSolder, symbol Device:R
Connections:
- net +BATT: now also U1.3 (OUT+), Q1.3 (D)
- net GND: now also R2.1, R5.1, R5.2, R6.1, R6.2; no longer BT1.2 (-), U1.6 (BAT-)
- net VBUS: now also D1.2 (A), Q1.1 (G), R2.2, R4.1, R4.2
- net at SW1.2 (B): now also D1.1 (K), Q1.2 (S); no longer U1.3 (OUT+)
- new net -BATT: BT1.2 (-), R3.1, R3.2, U1.6 (BAT-)
Other:
- moved on the sheet: C1, C2, C4, C5, SW1, U2, U3
